File: hardware/boards/glasgow/glasgow.sch (KiCad schematic (older format))
At the start: 77 parts, among them J1 USB_B_Micro, J4 Conn_01x02, U1 CY7C68013A-56LTX, U15 TPD3S014, U2 CAT24M01W, U3 CAT24C256W, U4 ICE40UP5K-SG48ITR, U7 LM3880MF-1AF, U8 MIC5355-S4YMME, Y1 24M

Commit message: revC WIP PCB work
Parts:
- removed R30: 100, Resistor_SMD:R_0603_1608Metric_Pad0.99x1.00mm_HandSolder, symbol Device:R
- removed unit 4 of U4
- added C76, C80: 4u7, Capacitor_SMD:C_0603_1608Metric_Pad1.05x0.95mm_HandSolder, symbol Device:C
- added C77, C78, C79, C81: u1, Capacitor_SMD:C_0402_1005Metric, symbol Device:C
- added R31, R32: 100, Resistor_SMD:R_0603_1608Metric_Pad1.05x0.95mm_HandSolder, symbol Device:R
- added U30: ICE40HX8K-BG121, Package_BGA:BGA-121_9.0x9.0mm_Layout11x11_P0.8mm_Ball0.4mm_Pad0.35mm_NSMD, symbol FPGA_Lattice:ICE40HX8K-BG121
- C1, C11, C12, C14, C16, C19, C26, C27, C28: footprint Capacitor_SMD:C_0603_1608Metric_Pad0.99x1.00mm_HandSolder -> Capacitor_SMD:C_0603_1608Metric_Pad1.05x0.95mm_HandSolder
- C10, C13, C15, C17, C2, C20, C21, C22, C23, C24, C25, C3, C33, C4, C5, C6, C7, C8, C9: footprint Capacitor_SMD:C_0603_1608Metric_Pad0.99x1.00mm_HandSolder -> Capacitor_SMD:C_0402_1005Metric
- C18: value 4u7 -> u1; footprint Capacitor_SMD:C_0603_1608Metric_Pad0.99x1.00mm_HandSolder -> Capacitor_SMD:C_0402_1005Metric; MPN LMK107BJ475KAHT -> TMK107BJ154KA-T
- R1, R10, R11, R12, R13, R14, R15, R16, R17, R18, R19, R2, R3, R4, R5, R6, R7, R8, R9: footprint Resistor_SMD:R_0603_1608Metric_Pad0.99x1.00mm_HandSolder -> Resistor_SMD:R_0603_1608Metric_Pad1.05x0.95mm_HandSolder
Connections:
- net labels added: GNDPLL0, GNDPLL1, VCCPLL0, VCCPLL1, VIO_AUX, Z0_N, Z0_P, Z10_N, Z10_P, Z11_N, Z11_P, Z12_N, Z12_P, Z1_N, Z1_P, Z2_N, Z2_P, Z3_N, Z3_P, Z4_N, Z4_P, Z5_N, Z5_P, Z6_N, Z6_P, Z7_N, Z7_P, Z8_N, Z8_P, Z9_N, Z9_P
- net labels removed: VCCPLL
- wire segments 393 -> 441

Commit message: revC: FX2<->FPGA routing take 1
Parts:
- removed R11: 100k, Resistor_SMD:R_0603_1608Metric_Pad1.05x0.95mm_HandSolder, symbol Device:R
- removed unit 2 of U4
- removed unit 3 of U4
- C11, C12: footprint Capacitor_SMD:C_0603_1608Metric_Pad1.05x0.95mm_HandSolder -> Capacitor_SMD:C_0402_1005Metric
- R1, R10, R12, R13, R14, R15, R16, R17, R18, R19, R2, R3, R31, R32, R4, R5, R6, R7, R8, R9: footprint Resistor_SMD:R_0603_1608Metric_Pad1.05x0.95mm_HandSolder -> Resistor_SMD:R_0402_1005Metric
Connections:
- wire segments 441 -> 410
Other:
- note removed: "Alternate use for\nFLAGD pin: INT1"
- note removed: "Imax @ 3V3 = 312 mA (all banks)"

Commit message: revC: delete old FPGA
No useful information left, since it's mostly just the port routing
remaining
Parts:
- removed U4: ICE40UP5K-SG48ITR, Package_DFN_QFN:QFN-48-1EP_7x7mm_P0.5mm_EP5.15x5.15mm, symbol FPGA_Lattice:ICE40UP5K-SG48ITR
Changed lines of the file:
@@
 Text Label 3950 4050 0    50   ~ 0
 CLKIF
-$Comp
-L FPGA_Lattice:ICE40UP5K-SG48ITR U4
-U 1 1 5ADBCDAC
-P 7250 3100
-F 0 "U4" H 6950 4150 50  0000 L CNN
-F 1 "ICE40UP5K-SG48ITR" H 6750 1950 50  0000 L CNN
-F 2 "Package_DFN_QFN:QFN-48-1EP_7x7mm_P0.5mm_EP5.15x5.15mm" H 7250 2050 50  0001 C CNN
-F 3 "http://www.latticesemi.com/Products/FPGAandCPLD/iCE40Ultra" H 6850 4100 50  0001 C CNN
-F 4 "Lattice" H 7250 3100 50  0001 C CNN "Mfg"
-F 5 "ICE40UP5K-SG48ITR50" H 7250 3100 50  0001 C CNN "MPN"
-	1    7250 3100
-	-1   0    0    -1
-$EndComp
 Entry Wire Line
 	6550 2450 6650 2550

Commit message: revC: route missing D0 and D1
Connections:
- wire segments 410 -> 412
Changed lines of the file:
@@
 Text Label 6200 4150 0    50   ~ 0
 D6
-Text Label 6800 3350 0    50   ~ 0
+Text Label 6200 3650 0    50   ~ 0
 D1
-Text Label 6750 3700 0    50   ~ 0
+Text Label 6200 3750 0    50   ~ 0
 D0
 Entry Wire Line
@@
 Wire Wire Line
 	4550 5200 4550 5500
+Entry Wire Line
+	6550 3650 6650 3750
+Entry Wire Line
+	6550 3750 6650 3850
+Wire Wire Line
+	6200 3650 6550 3650
+Wire Wire Line
+	6200 3750 6550 3750
 Wire Bus Line
 	4350 6250 6650 6250
@@
 	8000 2600 8000 4800
 Wire Bus Line
-	4350 2150 4350 6250
+	9650 2400 9650 4800
 Wire Bus Line
 	6650 2550 6650 6250
 Wire Bus Line
-	9650 2400 9650 4800
+	4350 2150 4350 6250
 $EndSCHEMATC

Commit message: revC: fix connector placement, LVDS connector testing
Parts:
- added J5: Conn_02x24_Odd_Even, Connector_PinHeader_1.27mm:PinHeader_2x24_P1.27mm_Vertical_SMD, symbol Connector_Generic:Conn_02x24_Odd_Even
Changed lines of the file:
@@
 Wire Bus Line
 	4350 2150 4350 6250
+$Comp
+L Connector_Generic:Conn_02x24_Odd_Even J5
+U 1 1 5D3E6DA7
+P 16850 4300
+F 0 "J5" H 16900 5617 50  0000 C CNN
+F 1 "Conn_02x24_Odd_Even" H 16900 5526 50  0000 C CNN
+F 2 "Connector_PinHeader_1.27mm:PinHeader_2x24_P1.27mm_Vertical_SMD" H 16850 4300 50  0001 C CNN
+F 3 "~" H 16850 4300 50  0001 C CNN
+	1    16850 4300
+	1    0    0    -1
+$EndComp
 $EndSCHEMATC

Commit message: revC: route LVDS
Parts:
- J5: value Conn_02x24_Odd_Even -> Conn_02x22_Odd_Even; footprint Connector_PinHeader_1.27mm:PinHeader_2x24_P1.27mm_Vertical_SMD -> Connector_PinHeader_1.27mm:PinHeader_2x22_P1.27mm_Vertical_SMD; symbol Connector_Generic:Conn_02x24_Odd_Even -> Connector_Generic:Conn_02x22_Odd_Even
Connections:
- wire segments 412 -> 449
Changed lines of the file:
@@
 Text Label 17550 5300 0    50   ~ 0
 Z10_N
-Text Label 17550 5400 0    50   ~ 0
+Text Label 15950 3500 2    50   ~ 0
 Z11_P
 Text Label 17550 5500 0    50   ~ 0
@@
 Wire Wire Line
 	6200 3750 6550 3750
+$Comp
+L Connector_Generic:Conn_02x22_Odd_Even J5
+U 1 1 5D3E6DA7
+P 16150 4300
+F 0 "J5" H 16200 5517 50  0000 C CNN
+F 1 "Conn_02x22_Odd_Even" H 16200 5426 50  0000 C CNN
+F 2 "Connector_PinHeader_1.27mm:PinHeader_2x22_P1.27mm_Vertical_SMD" H 16150 4300 50  0001 C CNN
+F 3 "~" H 16150 4300 50  0001 C CNN
+	1    16150 4300
+	1    0    0    -1
+$EndComp
+Wire Wire Line
+	15950 3300 15850 3300
+Wire Wire Line
+	15850 3300 15850 3600
+Wire Wire Line
+	16450 3300 16700 3300
+Wire Wire Line
+	16700 3300 16700 3100
+Wire Wire Line
+	16450 3400 16900 3400
+Wire Wire Line
+	16900 3400 16900 3100
+Wire Wire Line
+	16450 3500 17100 3500
+Wire Wire Line
+	17100 3500 17100 3100
+$Comp
+L power:+3.3V #PWR0102
+U 1 1 5D502274
+P 16900 3100
+F 0 "#PWR0102" H 16900 2950 50  0001 C CNN
+F 1 "+3.3V" H 16915 3273 50  0000 C CNN
+F 2 "" H 16900 3100 50  0001 C CNN
+F 3 "" H 16900 3100 50  0001 C CNN
+	1    16900 3100
+	-1   0    0    -1
+$EndComp
+$Comp
+L power:+1V2 #PWR0105
+U 1 1 5D5023DF
+P 17100 3100
+F 0 "#PWR0105" H 17100 2950 50  0001 C CNN
+F 1 "+1V2" H 17115 3273 50  0000 C CNN
+F 2 "" H 17100 3100 50  0001 C CNN
+F 3 "" H 17100 3100 50  0001 C CNN
+	1    17100 3100
+	-1   0    0    -1
+$EndComp
+$Comp
+L power:+5V #PWR0110
+U 1 1 5D50249A
+P 16700 3100
+F 0 "#PWR0110" H 16700 2950 50  0001 C CNN
+F 1 "+5V" H 16715 3273 50  0000 C CNN
+F 2 "" H 16700 3100 50  0001 C CNN
+F 3 "" H 16700 3100 50  0001 C CNN
+	1    16700 3100
+	-1   0    0    -1
+$EndComp
+Wire Wire Line
+	16450 3800 16550 3800
+Wire Wire Line
+	16550 3800 16550 4100
+Wire Wire Line
+	16550 5550 16200 5550
+$Comp
+L power:GND #PWR0114
+U 1 1 5D532335
+P 16200 5550
+F 0 "#PWR0114" H 16200 5300 50  0001 C CNN
+F 1 "GND" H 16205 5377 50  0000 C CNN
+F 2 "" H 16200 5550 50  0001 C CNN
+F 3 "" H 16200 5550 50  0001 C CNN
+	1    16200 5550
+	-1   0    0    -1
+$EndComp
+Connection ~ 16200 5550
+Wire Wire Line
+	16200 5550 15850 5550
+Wire Wire Line
+	16550 4100 16450 4100
+Connection ~ 16550 4100
+Wire Wire Line
+	16550 4100 16550 4400
+Wire Wire Line
+	16450 4400 16550 4400
+Connection ~ 16550 4400
+Wire Wire Line
+	16550 4400 16550 4700
+Wire Wire Line
+	16550 4700 16450 4700
+Connection ~ 16550 4700
+Wire Wire Line
+	16550 4700 16550 5000
+Wire Wire Line
+	16450 5000 16550 5000
+Connection ~ 16550 5000
+Wire Wire Line
+	16550 5000 16550 5300
+Wire Wire Line
+	16550 5300 16450 5300
+Connection ~ 16550 5300
+Wire Wire Line
+	16550 5300 16550 5550
+Wire Wire Line
+	15950 3600 15850 3600
+Connection ~ 15850 3600
+Wire Wire Line
+	15850 3600 15850 3900
+Wire Wire Line
+	15950 3900 15850 3900
+Connection ~ 15850 3900
+Wire Wire Line
+	15850 3900 15850 4200
+Wire Wire Line
+	15950 4200 15850 4200
+Connection ~ 15850 4200
+Wire Wire Line
+	15850 4200 15850 4500
+Wire Wire Line
+	15950 4500 15850 4500
+Connection ~ 15850 4500
+Wire Wire Line
+	15850 4500 15850 4800
+Wire Wire Line
+	15950 4800 15850 4800
+Connection ~ 15850 4800
+Wire Wire Line
+	15850 4800 15850 5100
+Wire Wire Line
+	15950 5100 15850 5100
+Connection ~ 15850 5100
+Wire Wire Line
+	15850 5100 15850 5400
+Wire Wire Line
+	15950 5400 15850 5400
+Connection ~ 15850 5400
+Wire Wire Line
+	15850 5400 15850 5550
+Text Label 16900 5400 2    50   ~ 0
+VIO_AUX
+Wire Wire Line
+	16450 5400 16900 5400
 Wire Bus Line
 	4350 6250 6650 6250
@@
 Wire Bus Line
 	4350 2150 4350 6250
-$Comp
-L Connector_Generic:Conn_02x24_Odd_Even J5
-U 1 1 5D3E6DA7
-P 16850 4300
-F 0 "J5" H 16900 5617 50  0000 C CNN
-F 1 "Conn_02x24_Odd_Even" H 16900 5526 50  0000 C CNN
-F 2 "Connector_PinHeader_1.27mm:PinHeader_2x24_P1.27mm_Vertical_SMD" H 16850 4300 50  0001 C CNN
-F 3 "~" H 16850 4300 50  0001 C CNN
-	1    16850 4300
-	1    0    0    -1
-$EndComp
+Text Label 16450 3600 0    50   ~ 0
+Z12_P
+Text Label 16450 3700 0    50   ~ 0
+Z12_N
+Text Label 16450 3900 0    50   ~ 0
+Z9_N
+Text Label 16450 4000 0    50   ~ 0
+Z9_P
+Text Label 16450 4200 0    50   ~ 0
+Z7_N
+Text Label 16450 4300 0    50   ~ 0
+Z7_P
+Text Label 16450 4500 0    50   ~ 0
+Z5_N
+Text Label 16450 4600 0    50   ~ 0
+Z5_P
+Text Label 16450 4800 0    50   ~ 0
+Z4_P
+Text Label 16450 4900 0    50   ~ 0
+Z4_N
+Text Label 16450 5100 0    50   ~ 0
+Z1_N
+Text Label 16450 5200 0    50   ~ 0
+Z1_P
+Text Label 15950 5300 2    50   ~ 0
+Z0_N
+Text Label 15950 5200 2    50   ~ 0
+Z0_P
+Text Label 15950 5000 2    50   ~ 0
+Z2_P
+Text Label 15950 4900 2    50   ~ 0
+Z2_N
+Text Label 15950 4700 2    50   ~ 0
+Z3_N
+Text Label 15950 4600 2    50   ~ 0
+Z3_P
+Text Label 15950 4400 2    50   ~ 0
+Z6_N
+Text Label 15950 4300 2    50   ~ 0
+Z6_P
+Text Label 15950 4100 2    50   ~ 0
+Z8_N
+Text Label 15950 4000 2    50   ~ 0
+Z8_P
+Text Label 15950 3800 2    50   ~ 0
+Z10_N
+Text Label 15950 3700 2    50   ~ 0
+Z10_P
+Text Label 17550 5400 0    50   ~ 0
+Z11_P
+Text Label 15950 3400 2    50   ~ 0
+Z11_N
 $EndSCHEMATC
