File: hardware/boards/glasgow/glasgow.kicad_pcb (KiCad board)
At the start: 4 copper layers, 80 x 49 mm, 240 parts, among them J1 USB_B_Micro, J10 Conn_01x03, J2 Conn_02x10_Odd_Even, J3 Conn_02x10_Odd_Even, J4 Conn_01x02, J5 Conn_02x22_Odd_Even, J6 Conn_01x08, J7 Conn_01x08, J8 Conn_01x08, J9 Conn_01x08, U1 CY7C68013A-56LTX, U10 SN74LVC1T45DRL, U11 SN74LVC1T45DRL, U12 ADC081C021CIMM, U13 DAC081C081CIMK, U14 TPS73101DBV, U15 TPD3S014, U16 SN74LVC1T45DRL, U17 SN74LVC1T45DRL, U18 SN74LVC1T45DRL, U19 PCA6408APW, U2 CAT24M01W, U20 DAC081C081CIMK, U21 ADC081C021CIMM, U22 SN74LVC1T45DRL, U23 SN74LVC1T45DRL, U24 SN74LVC1T45DRL, U25 SN74LVC1T45DRL, U26 SN74LVC1T45DRL, U27 SN74LVC1T45DRL, U28 SN74LVC1T45DRL, U29 SN74LVC1T45DRL, U3 CAT24C256W, U30 ICE40HX8K-BG121, U31 TPS73101DBV, U32 SN74LVC1T45DRL, U33 MG2040, U34 ATECC508A, U35 MG2040, U36 TLV73312PQDRVRQ1, U4 SN74LVC1T45DRL, U5 PCA6408APW, U6 SN74LVC1T45DRL, U7 LM3880MF-1AF, U8 TLV75533PDRVR, U9 SN74LVC1T45DRL, Y1 24M

Commit message: refilled zones and revC1 jlc
Other:
- board text added: "JLCJLCJLCJLCJLC"
